Commit message: Initial upload

File: src/rham_description/urdf/rham_bot.urdf (robot description, URDF)
Before this commit: robot rham_bot, 5 links, 4 joints
Joints:
- joint caster_link_jt: type continuous -> fixed

File: src/rham_description/xacro/gazebo/plugin/plugin.xacro (robot description, xacro)
@@ -8,4 +8,26 @@
             </plugin>
         </gazebo>
+        <gazebo>
+            <plugin name="differential_drive_controller" filename="libgazebo_ros_diff_drive.so">
+                <!-- info -->
+                <leftJoint>left_motor_link_jt</leftJoint>
+                <rightJoint>right_motor_link_jt</rightJoint>
+                <wheelSeparation>0.234</wheelSeparation>
+                <wheelDiameter>0.065</wheelDiameter>
+                <!-- speed -->
+                <wheelAcceleration>1.0</wheelAcceleration>
+                <max_wheel_acceleration>10.0</max_wheel_acceleration>
+                <wheelTorque>3</wheelTorque>
+                <!-- node -->
+                <commandTopic>cmd_vel</commandTopic>
+                <odometryTopic>odom</odometryTopic>
+                <odometryFrame>odom</odometryFrame>
+                <publishOdom>true</publishOdom>
+                <robotBaseFrame>basefoot_link</robotBaseFrame>
+                <odometrySource>1</odometrySource>
+                <publishWheelTF>true</publishWheelTF>
+                <publishWheelJointState>true</publishWheelJointState>
+            </plugin>
+        </gazebo>
     </xacro:macro>
 </robot>

File: src/rham_description/xacro/gazebo/wheel/wheel.xacro (robot description, xacro)
@@ -15,6 +15,6 @@
         </gazebo>
         <gazebo reference="caster_link">
-            <mu1>1.5</mu1>
-            <mu2>1.5</mu2>
+            <mu1>0.001</mu1>
+            <mu2>0.001</mu2>
             <selfCollide>true</selfCollide>
             <material>Gazebo/Green</material>
